File: Any-Screen-Touch-Screen_AnchorMod/Any-Screen-Touch-Screen_AnchorMod.kicad_sch (KiCad schematic)
At the start: 28 parts, among them P1 USB_C_Plug_USB2.0, Q2 S8050, Q3 S8050, SW1 SW_Push, SW2 SW_Push, U1 ESP32-S3-WROOM-1, U2 CP2104

Commit message: pen firmware prog, update on anchor looping
Connections:
- net EXT_ON: now also U1.38 (IO2); no longer U1.5 (IO5)
- net INT: now also U1.39 (IO1); no longer U1.4 (IO4)
- net RESET_ACT_L: now also U1.5 (IO5); no longer U1.7 (IO7)
- net WAKEUP: now also U1.4 (IO4); no longer U1.6 (IO6)

Commit message: updated pcb design
Parts:
- removed D1, D2, D3, D4: LED, symbol Device:LED
- removed Q2, Q3: S8050, Package_TO_SOT_THT:TO-92_Inline, symbol Transistor_BJT:S8050
- removed SW1, SW2: SW_Push, symbol Switch:SW_Push
- added C5: 1 μF, Capacitor_SMD:C_0805_2012Metric_Pad1.18x1.45mm_HandSolder, symbol Device:C
- added C6: 10 μF, Capacitor_SMD:C_0805_2012Metric_Pad1.18x1.45mm_HandSolder, symbol Device:C
- added C7: 33 μF, Capacitor_SMD:C_0805_2012Metric_Pad1.18x1.45mm_HandSolder, symbol Device:C
- added C8: 0.47 μF, Capacitor_SMD:C_0805_2012Metric_Pad1.18x1.45mm_HandSolder, symbol Device:C
- added C9: 1uF, Capacitor_SMD:C_0805_2012Metric_Pad1.18x1.45mm_HandSolder, symbol Device:C_Small
- added H1, H2, H3, H4: MountingHole, MountingHole:MountingHole_3.2mm_M3, symbol Mechanical:MountingHole
- added J1: Reset button, Connector_Molex:Molex_KK-254_AE-6410-02A_1x02_P2.54mm_Vertical, symbol Connector_Generic:Conn_01x02
- added J2: Flash button, Connector_Molex:Molex_KK-254_AE-6410-02A_1x02_P2.54mm_Vertical, symbol Connector_Generic:Conn_01x02
- added J3: Power Switch, Connector_Molex:Molex_KK-254_AE-6410-02A_1x02_P2.54mm_Vertical, symbol Connector_Generic:Conn_01x02
- added J4: Battery Terminals, Connector_Molex:Molex_KK-254_AE-6410-02A_1x02_P2.54mm_Vertical, symbol Connector_Generic:Conn_01x02
- added J5: LED1, Connector_Molex:Molex_KK-254_AE-6410-02A_1x02_P2.54mm_Vertical, symbol Connector_Generic:Conn_01x02
- added J6: LED2, Connector_Molex:Molex_KK-254_AE-6410-02A_1x02_P2.54mm_Vertical, symbol Connector_Generic:Conn_01x02
- added J7: LED3, Connector_Molex:Molex_KK-254_AE-6410-02A_1x02_P2.54mm_Vertical, symbol Connector_Generic:Conn_01x02
- added J8: LED4, Connector_Molex:Molex_KK-254_AE-6410-02A_1x02_P2.54mm_Vertical, symbol Connector_Generic:Conn_01x02
- added L2: MSS5131-222MLB, footprints:IND_MSS5131_COC, symbol CoilCraft Inductor MSS:MSS5131-222MLB
- added R13, R14, R15: 10kΩ, Resistor_SMD:R_0805_2012Metric_Pad1.20x1.40mm_HandSolder, symbol Device:R
- added R16: 10k, Resistor_SMD:R_0805_2012Metric_Pad1.20x1.40mm_HandSolder, symbol Device:R
- added TP1, TP2, TP3: TestPoint, TestPoint:TestPoint_Keystone_5010-5014_Multipurpose, symbol Connector:TestPoint
- added U3: BQ27441-G1, Package_SON:Texas_S-PDSO-N12, symbol Battery_Management:BQ27441-G1
- added U5: TPS63001, Package_SON:Texas_DRC0010J_ThermalVias, symbol Regulator_Switching:TPS63001
- C1, C2, C3, C4: footprint (none) -> Capacitor_SMD:C_0805_2012Metric_Pad1.18x1.45mm_HandSolder
- P1: footprint (none) -> Connector_USB:USB_C_Plug_Molex_105444
- R1, R10, R2, R3, R4, R5, R6, R7, R8, R9: footprint (none) -> Resistor_SMD:R_0805_2012Metric_Pad1.20x1.40mm_HandSolder
- R11: value 1k -> 10kΩ; footprint (none) -> Resistor_SMD:R_0805_2012Metric_Pad1.20x1.40mm_HandSolder
- R12: value 1k -> 10mΩ; footprint (none) -> Resistor_SMD:R_0805_2012Metric_Pad1.20x1.40mm_HandSolder
- U2: footprint Package_DFN_QFN:QFN-24-1EP_4x4mm_P0.5mm_EP2.6x2.6mm -> Package_DFN_QFN:QFN-24-1EP_4x4mm_P0.5mm_EP2.7x2.7mm_ThermalVias
Connections:
- net +3.3V: now also C7.1, R13.1, R14.1, R15.1, TP1.1, U5.1 (VOUT), U5.10 (FB)
- net EN_FLASH: now also R9.2; no longer R9.1
- net EXT_ON: now also U1.5 (IO5); no longer U1.38 (IO2)
- net GND: now also R11.1, C5.2, C6.1, C7.2, C8.2, C9.1, J1.2 (Pin_2), J2.2 (Pin_2), J4.2 (Pin_2), J5.2 (Pin_2), J6.2 (Pin_2), J7.2 (Pin_2), J8.2 (Pin_2), R16.1, U3.3 (V_{SS}), U5.11 (PGND), U5.3 (PGND), U5.9 (GND)
- net INT: now also U1.4 (IO4); no longer U1.39 (IO1)
- net RESET_ACT_L: now also U1.7 (IO7); no longer U1.5 (IO5)
- net RESET_ESP: now also C9.2, J1.1 (Pin_1), R15.2
- net USB_READY: no longer R11.1
- net USB_SEND: no longer R12.1
- net WAKEUP: now also U1.6 (IO6); no longer U1.4 (IO4)
- net at R7.1: now also J7.1 (Pin_1)
- net MCU GPIO: now reaches U1.23 (IO21)
- net MCU GPIO: now also U3.12 (GPOUT)
- net at R5.1: now also J5.1 (Pin_1)
- net at R8.1: now also J8.1 (Pin_1)
- net at R12.2: now also C6.2, U3.7 (SRN), U5.5 (VIN), U5.6 (EN), U5.7 (PS/SYNC), U5.8 (VINA)
- net at R11.2: now also U3.10 (BIN)
- net at R6.1: now also J6.1 (Pin_1)
- net at P1.B5 (VCONN): now also R16.2
- new net: C8.1, U3.5 (V_{DD})
- new net: C5.1, J3.2 (Pin_2), R12.1, U3.6 (BAT), U3.8 (SRP)
- new net: J2.1 (Pin_1), R9.1
- new net: J3.1 (Pin_1), J4.1 (Pin_1)
- new net: L2.1, TP2.1, U5.2 (L2)
- new net: L2.2, TP3.1, U5.4 (L1)
- new net I2C Clock: R13.2, U1.38 (IO2), U3.2 (SCL)
- new net I2C Data: R14.2, U1.39 (IO1), U3.1 (SDA)
Other:
- note added: "3.3V Buck Converter"
- note added: "Battery Fuel Gauge"
- note added: "Microcontroller"
- note added: "USB-to-UART"
- moved on the sheet: C1, C2, C3, C4, DWM1, P1, R1, R10, R2, R3, R4, R5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
